File: MM_Main_new.sch (EAGLE design)
At the start: 37 parts, among them IC1 FXAS21002C, Q1 TEFT4300, Q2 TEFT4300, Q3 TEFT4300, Q4 TEFT4300, Q5 IRF7101, Q6 IRF7101

Commit message: gitignore i sch
Parts:
- removed C_CRYS1, C_CRYS2: 27p, rcl:C-EUC0805
- removed Q5, Q6: IRF7101, _microMouse:IRF7101
- added BT, PROG: (no value), pinhead:PINHD-1X4
- added C11, C15: tant-a-100u, rcl:CPOL-EUSMCA
- added C12, C18: 100n, rcl:C-EUC0603
- added C13, C22: tant-a-10u, rcl:CPOL-EUSMCA
- added C14: 100n, rcl:C-EUC0805
- added C16, C21: tant-a-4,7u, rcl:CPOL-EUSMCA
- added C_OSC1, C_OSC2: 27p, rcl:C-EUC0805
- added C_OSC3, C_OSC4: 10p, rcl:C-EUC0805
- added D1, D2, D3, D4: SFH4545, _microMouse:SFH4545
- added F1: (no value), fuse:GSH15
- added IC2: TB6612FNG, _microMouse:TB6612FNG
- added IC3: FXAS21002C, _microMouse:FXAS21002C
- added IC4: LD117ADT50TR, v-reg:LD117ADT50TR
- added LED1, LED2: (no value), led:LEDSML1206
- added M_L, M_R, ZAS: (no value), pinhead:PINHD-1X3
- added Q8: 32,768kHz, crystal:CRYSTALHC49U70
- added R12, R13, R16: 10K, resistor:R-EU_R0805
- added R14, R15: 47k, resistor:R-EU_R0805
- added U$4: MCP1825, _microMouse:MCP1825
- C10: value 4,7u -> 100n; device rcl:C-EUC3216 -> rcl:C-EUC0603
- C6: value 4,7u -> tant-a-10u; device rcl:C-EUC3216 -> rcl:CPOL-EUSMCA
- C8: value 100n -> tant-a-4u7; device rcl:C-EUC0603 -> rcl:CPOL-EUSMCA
- IC1: value FXAS21002C -> ULN2003AD; device _microMouse:FXAS21002C -> uln-udn:ULN2003AD
- Q7: value (none) -> 8MHz
- R10: value 47k -> 10k; device rcl:R-EU_R0805 -> resistor:R-EU_R0805
- R11: value (none) -> 10K; device rcl:R-EU_R0805 -> resistor:R-EU_R0805
- R9: value 47k -> (none)
- U$3: value MCP1825 -> TACTILE-SWITCH-7914G; device _microMouse:MCP1825 -> GeekAmmo:TACTILE-SWITCH-7914G
Connections:
- net N$5 renamed CS_G
- net N$8 renamed INT_G
- removed net 3V3: Q1.C, Q2.C, Q3.C, Q4.C, U$3.OUT
- removed net BOOT1: R10.1
- removed net L: Q2.E, R2.2
- removed net L_PRZOD: Q1.E, R1.2
- removed net MOS_L: Q5B.G
- removed net MOS_L_PRZOD: Q5A.G
- removed net MOS_R: Q6A.G
- removed net MOS_R_PRZOD: Q6B.G
- removed net N$22: IC1.INT1
- removed net N$23: IC1.RST_B, R11.1
- removed net N$3: C3.1, U$2.VDDIO
- removed net R: Q3.E, R3.2
- removed net R_PRZOD: Q4.E, R4.2
- new net +3V3: BT.4, C12.1, C13.+, C18.1, C3.1, C4.2, C5.+, C8.+, IC2.STBY, IC2.VCC, PROG.1, Q1.C, Q2.C, Q3.C, Q4.C, R10.2, R12.2, R13.2, R16.2, R9.2, U$1.VBAT, U$2.VDD, U$2.VDDIO, U$4.OUT
- new net +7V: C11.+, C15.+, C6.+, F1.2, IC2.VM1, IC2.VM2, IC2.VM3, R5.2, R6.2, R7.2, R8.2
- new net ADC_L: Q2.E, R2.2, U$1.PA2
- new net ADC_LF: Q1.E, R1.2, U$1.PA1
- new net ADC_R: Q3.E, R3.2, U$1.PA3
- new net ADC_RF: Q4.E, R4.2, U$1.PA4
- new net BT_RXD: BT.1, U$1.PA9
- new net BT_TXD: BT.2, U$1.PA10
- new net BUTTON: R11.1, U$1.PA0-WKUP
- new net D_L: IC1.I3, IC1.I4, U$1.PB1
- new net D_LF: IC1.I1, IC1.I2, U$1.PB0
- new net D_R: IC1.I5, IC1.I6, U$1.PB10
- new net D_RF: IC1.I7, U$1.PB11
- new net GNDA: C11.-, C15.-, IC2.PGND1, IC2.PGND1', IC2.PGND2, IC2.PGND2', ZAS.1, ZAS.3
- new net LED: LED2.C
- new net LED1: U$1.PB9
- new net LED2: U$1.PB8
- new net MISO: IC3.SA0/MISO, U$1.PB14, U$2.SA0/MISO
- new net MOSI: IC3.SDA/MOSI, U$1.PB15, U$2.SDA/MOSI
- new net M_L_IN1: IC2.AIN2, U$1.PB5
- new net M_L_IN2: IC2.AIN1, U$1.PB4
- new net M_L_PWM: IC2.PWMA, U$1.PB7
- new net M_R_IN1: IC2.BIN1, U$1.PB3
- new net M_R_IN2: IC2.BIN2, U$1.PA15
- new net M_R_PWM: IC2.PWMB, U$1.PB6
- new net N$26: C10.1, IC3.VREGD
- new net N$27: IC3.PWR_CTRL
- new net N$28: IC3.INT1
- new net N$29: R11.2, U$3.1
- new net N$30: IC3.RST_B, R9.1
- new net N$31: R14.1, U$1.BOOT0
- new net N$33: R15.2, U$1.PB2
- new net OSC32_IN: C_OSC3.2, Q8.2, U$1.PC14-OSC32_IN
- new net OSC32_OUT: C_OSC4.2, Q8.1, U$1.PC15-OSC_OUT
- new net OSC_IN: C_OSC1.2, Q7.2, U$1.PD0-OSC_IN
- new net OSC_OUT: C_OSC2.2, Q7.1, U$1.PD1-OSC_OUT
- new net SCK: U$1.PB13
- new net SCLK: IC3.SCL/SCLK, U$2.SCL/SCLK
- new net SWCLK: PROG.4, U$1.PA14
- new net SWDIO: PROG.3, U$1.PA13
- new net VBAT: C22.+, IC4.IN, U$3.3
- new net VDDA: C14.2, C16.-, U$1.VDDA
- new net VSSA: C14.1, C16.+, U$1.VSSA
- net 5V: now also C21.+, IC4.OUT, U$4.IN, U$4.SHDN; no longer C6.1, U$3.IN, U$3.SHDN
- net GND: now also BT.3, C10.2, C12.2, C13.-, C21.-, C22.-, C6.-, C9.1, C_OSC1.1, C_OSC2.1, C_OSC3.1, C_OSC4.1, IC1.GND, IC2.GND, IC3.GND1, IC3.GND2, IC3.GND4, IC3.RGND, IC3.RGND1, IC3.RGND2, IC3.RGND3, IC3.RGND4, IC3.RGND5, IC3.RGND6, IC3.RGND7, IC3.RGND8, IC4.ADJ, LED1.C, PROG.2, R14.2, R15.1, U$4.GND; no longer C8.2, IC1.GND1, IC1.GND2, IC1.GND4, IC1.RGND, IC1.RGND1, IC1.RGND2, IC1.RGND3, IC1.RGND4, IC1.RGND5, IC1.RGND6, IC1.RGND7, IC1.RGND8, Q5A.S, Q5B.S, Q6A.S, Q6B.S, R9.2
- net GND3: now also C18.2, C8.-, IC3.GND3; no longer C10.2, C9.2, IC1.GND3
- net N$1: now also R16.1, U$4.PWRGD; no longer U$2.SDA/MOSI
- net N$10: now also D2.A, R6.1; no longer C6.2, U$3.GND
- net N$11: now also D3.A, R7.1; no longer U$1.VSSA
- net N$12: now also D4.A, R8.1; no longer U$1.VDDA
- net N$13: now also D1.C, IC1.O1, IC1.O2; no longer R10.2, U$1.PB2
- net N$14: now also D2.C, IC1.O3, IC1.O4; no longer U$3.PWRGD
- net N$15: now also D3.C, IC1.O5, IC1.O6; no longer IC1.SDA/MOSI
- net N$16: now also D4.C, IC1.O7; no longer IC1.SCL/SCLK
- net N$17: now also LED1.A, R12.1; no longer IC1.SA0/MISO
- net N$18: now also IC2.AO2, IC2.AO2', M_L.2; no longer C_CRYS1.2, Q7.2
- net N$19: now also IC2.BO2, IC2.BO2', M_R.1, M_R.3; no longer IC1.SPI_CS_B
- net N$2: now also C7.2, R10.1, U$1.NRST; no longer U$2.SA0/MISO
- net N$20: now also IC2.BO1, IC2.BO1', M_R.2; no longer C8.1, IC1.VREGD
- net N$21: now also LED2.A, R13.1; no longer IC1.PWR_CTRL
- net N$24: now also F1.1, ZAS.2; no longer C_CRYS2.2, Q7.1
- net N$25: now also IC3.SPI_CS_B; no longer C_CRYS1.1, C_CRYS2.1
- net N$4: now also D1.A, R5.1; no longer R9.1, U$1.BOOT0
- net N$9: now also IC2.AO1, IC2.AO1', M_L.1, M_L.3; no longer U$2.SCL/SCLK
- net VCC: now also IC3.I2C_B/SPI; no longer C4.2, C5.+, IC1.I2C_B/SPI, R11.2, R5.2, R6.2, R7.2, R8.2, U$2.VDD
- net VDD: now also IC3.VDD; no longer C10.1, C9.1, IC1.VDD
- net VDD1: no longer U$1.VDD_1
- net VDD2: no longer U$1.VDD_2
- net VDD3: no longer U$1.VDD_3
- net VDDIO: now also C9.2, IC3.VDDIO; no longer C7.2, IC1.VDDIO
- net VSS1: no longer U$1.VSS_1
- net VSS2: no longer U$1.VSS_2
- net VSS3: no longer U$1.VSS_3
Other:
- note added: "Boot1 Boot0 x0 - main flash memory 10 - bootloader 11 - SRAM"
- note added: "C8T6"
- note added: "DO ENKODEROW"
- note added: "ZMIENIC OBUDOWE KWARCU Q8"
- moved on the sheet: C10, C7, C9, C_V1, C_V2, C_V3, Q7, R10, R11, R9
