File: MM_Main_old.sch (EAGLE design)
At the start: 47 parts, among them IC1 FXAS21002C, Q1 TEFT4300, Q2 TEFT4300, Q3 TEFT4300, Q4 TEFT4300, Q5 IRF7101, Q6 IRF7101, Q7 8MHz, Q8 32,768kHz

Commit message: gitignore i sch
Connections:
- new net N$27: D4.A, R8.1
- new net N$28: D3.A, R7.1
- new net N$29: D2.A, R6.1
- new net N$30: D1.A, R5.1
- net 5V: no longer R5.2, R6.2, R7.2, R8.2
- net N$11: now also D1.C, Q5A.D; no longer R5.1
- net N$12: now also D2.C, Q5B.D; no longer R6.1
- net N$25: now also D3.C, Q6A.D; no longer R7.1
- net N$26: now also D4.C, Q6B.D; no longer R8.1
- net VCC: now also R5.2, R6.2, R7.2, R8.2
Other:
- note added: "5V STABILIZATOR"
- moved on the sheet: D1, D2, D3, D4, Q6B, R5, R6, R7, R8
Changed lines of the file:
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@@
 <text x="391.16" y="40.64" size="1.778" layer="90">VDDIO (1.62 to VDD + 0.3 V)</text>
 <text x="-88.9" y="-58.42" size="1.778" layer="97">ZMIENIC OBUDOWE KWARCU Q8</text>
+<text x="87.63" y="12.7" size="1.778" layer="97" rot="R90">5V STABILIZATOR</text>
 </plain>
 <instances>
@@
 <instance part="Q5" gate="B" x="93.98" y="127"/>
 <instance part="Q6" gate="A" x="114.3" y="127"/>
-<instance part="Q6" gate="B" x="134.62" y="127"/>
+<instance part="Q6" gate="B" x="137.16" y="127"/>
 <instance part="AGND1" gate="GND" x="104.14" y="116.84"/>
-<instance part="R5" gate="G$1" x="76.2" y="154.94" rot="R90"/>
-<instance part="R6" gate="G$1" x="96.52" y="154.94" rot="R90"/>
-<instance part="R7" gate="G$1" x="116.84" y="154.94" rot="R90"/>
-<instance part="R8" gate="G$1" x="139.7" y="154.94" rot="R90"/>
+<instance part="R5" gate="G$1" x="76.2" y="157.48" rot="R90"/>
+<instance part="R6" gate="G$1" x="96.52" y="157.48" rot="R90"/>
+<instance part="R7" gate="G$1" x="116.84" y="157.48" rot="R90"/>
+<instance part="R8" gate="G$1" x="139.7" y="157.48" rot="R90"/>
 <instance part="C_V1" gate="G$1" x="-73.66" y="25.4"/>
 <instance part="C_V2" gate="G$1" x="-81.28" y="25.4"/>
@@
 <instance part="GND15" gate="1" x="-88.9" y="48.26"/>
 <instance part="P+6" gate="VCC" x="-88.9" y="71.12"/>
-<instance part="D1" gate="G$1" x="76.2" y="142.24"/>
-<instance part="D2" gate="G$1" x="96.52" y="142.24"/>
-<instance part="D3" gate="G$1" x="116.84" y="142.24"/>
-<instance part="D4" gate="G$1" x="139.7" y="142.24"/>
-<instance part="5V" gate="G$1" x="101.6" y="167.64"/>
+<instance part="D1" gate="G$1" x="76.2" y="142.748"/>
+<instance part="D2" gate="G$1" x="96.52" y="144.018"/>
+<instance part="D3" gate="G$1" x="116.84" y="144.018"/>
+<instance part="D4" gate="G$1" x="139.7" y="144.018"/>
+<instance part="5V" gate="G$1" x="96.52" y="168.91"/>
 </instances>
 <busses>
@@
 <wire x1="96.52" y1="121.92" x2="96.52" y2="119.38" width="0.1524" layer="91"/>
 <pinref part="Q6" gate="B" pin="S"/>
-<wire x1="116.84" y1="119.38" x2="137.16" y2="119.38" width="0.1524" layer="91"/>
-<wire x1="137.16" y1="119.38" x2="137.16" y2="121.92" width="0.1524" layer="91"/>
+<wire x1="116.84" y1="119.38" x2="139.7" y2="119.38" width="0.1524" layer="91"/>
+<wire x1="139.7" y1="119.38" x2="139.7" y2="121.92" width="0.1524" layer="91"/>
 </segment>
 <segment>
@@
 <label x="-78.74" y="-78.74" size="1.27" layer="95" xref="yes"/>
 </segment>
+<segment>
+<pinref part="R5" gate="G$1" pin="2"/>
+<wire x1="76.2" y1="162.56" x2="76.2" y2="163.83" width="0.1524" layer="91"/>
+<pinref part="R6" gate="G$1" pin="2"/>
+<wire x1="76.2" y1="163.83" x2="96.52" y2="163.83" width="0.1524" layer="91"/>
+<wire x1="96.52" y1="163.83" x2="96.52" y2="162.56" width="0.1524" layer="91"/>
+<pinref part="R7" gate="G$1" pin="2"/>
+<wire x1="116.84" y1="162.56" x2="116.84" y2="163.83" width="0.1524" layer="91"/>
+<wire x1="116.84" y1="163.83" x2="96.52" y2="163.83" width="0.1524" layer="91"/>
+<junction x="96.52" y="163.83"/>
+<pinref part="R8" gate="G$1" pin="2"/>
+<wire x1="139.7" y1="162.56" x2="139.7" y2="163.83" width="0.1524" layer="91"/>
+<wire x1="139.7" y1="163.83" x2="116.84" y2="163.83" width="0.1524" layer="91"/>
+<junction x="116.84" y="163.83"/>
+<pinref part="5V" gate="G$1" pin="VCC"/>
+<wire x1="96.52" y1="166.37" x2="96.52" y2="163.83" width="0.1524" layer="91"/>
+</segment>
 </net>
 <net name="N$5" class="0">
@@
 <segment>
 <pinref part="Q5" gate="A" pin="G"/>
-<wire x1="68.58" y1="124.46" x2="58.42" y2="124.46" width="0.1524" layer="91"/>
+<wire x1="68.58" y1="124.46" x2="60.96" y2="124.46" width="0.1524" layer="91"/>
 <label x="53.34" y="121.92" size="1.778" layer="95"/>
 </segment>
@@
 <segment>
 <pinref part="Q6" gate="B" pin="G"/>
-<wire x1="129.54" y1="124.46" x2="121.92" y2="124.46" width="0.1524" layer="91"/>
+<wire x1="132.08" y1="124.46" x2="121.92" y2="124.46" width="0.1524" layer="91"/>
 <label x="119.38" y="121.92" size="1.778" layer="95"/>
 </segment>
@@
 <wire x1="96.52" y1="30.48" x2="91.44" y2="30.48" width="0.1524" layer="91"/>
 </segment>
-<segment>
-<wire x1="101.6" y1="165.1" x2="101.6" y2="162.56" width="0.1524" layer="91"/>
-<wire x1="101.6" y1="162.56" x2="96.52" y2="162.56" width="0.1524" layer="91"/>
-<wire x1="96.52" y1="162.56" x2="76.2" y2="162.56" width="0.1524" layer="91"/>
-<wire x1="101.6" y1="162.56" x2="116.84" y2="162.56" width="0.1524" layer="91"/>
-<wire x1="116.84" y1="162.56" x2="139.7" y2="162.56" width="0.1524" layer="91"/>
-<wire x1="139.7" y1="162.56" x2="139.7" y2="160.02" width="0.1524" layer="91"/>
-<wire x1="116.84" y1="162.56" x2="116.84" y2="160.02" width="0.1524" layer="91"/>
-<wire x1="96.52" y1="162.56" x2="96.52" y2="160.02" width="0.1524" layer="91"/>
-<wire x1="76.2" y1="162.56" x2="76.2" y2="160.02" width="0.1524" layer="91"/>
-<pinref part="R5" gate="G$1" pin="2"/>
-<pinref part="R6" gate="G$1" pin="2"/>
-<pinref part="R7" gate="G$1" pin="2"/>
-<pinref part="R8" gate="G$1" pin="2"/>
-<pinref part="5V" gate="G$1" pin="VCC"/>
-</segment>
 </net>
 <net name="N$14" class="0">
@@
 <net name="N$11" class="0">
 <segment>
+<pinref part="Q5" gate="A" pin="D"/>
+<pinref part="D1" gate="G$1" pin="C"/>
+<wire x1="76.2" y1="138.43" x2="76.2" y2="132.08" width="0.1524" layer="91"/>
+</segment>
+</net>
+<net name="N$12" class="0">
+<segment>
+<pinref part="Q5" gate="B" pin="D"/>
+<pinref part="D2" gate="G$1" pin="C"/>
+<wire x1="96.52" y1="139.7" x2="96.52" y2="132.08" width="0.1524" layer="91"/>
+</segment>
+</net>
+<net name="N$25" class="0">
+<segment>
+<pinref part="Q6" gate="A" pin="D"/>
+<pinref part="D3" gate="G$1" pin="C"/>
+<wire x1="116.84" y1="139.7" x2="116.84" y2="132.08" width="0.1524" layer="91"/>
+</segment>
+</net>
+<net name="N$26" class="0">
+<segment>
+<pinref part="Q6" gate="B" pin="D"/>
+<pinref part="D4" gate="G$1" pin="C"/>
+<wire x1="139.7" y1="139.7" x2="139.7" y2="132.08" width="0.1524" layer="91"/>
+</segment>
+</net>
+<net name="N$27" class="0">
+<segment>
+<pinref part="D4" gate="G$1" pin="A"/>
+<pinref part="R8" gate="G$1" pin="1"/>
+<wire x1="139.7" y1="152.4" x2="139.7" y2="147.32" width="0.1524" layer="91"/>
+</segment>
+</net>
+<net name="N$28" class="0">
+<segment>
+<pinref part="D3" gate="G$1" pin="A"/>
+<pinref part="R7" gate="G$1" pin="1"/>
+<wire x1="116.84" y1="152.4" x2="116.84" y2="147.32" width="0.1524" layer="91"/>
+</segment>
+</net>
+<net name="N$29" class="0">
+<segment>
+<pinref part="D2" gate="G$1" pin="A"/>
+<pinref part="R6" gate="G$1" pin="1"/>
+<wire x1="96.52" y1="152.4" x2="96.52" y2="147.32" width="0.1524" layer="91"/>
+</segment>
+</net>
+<net name="N$30" class="0">
+<segment>
+<pinref part="D1" gate="G$1" pin="A"/>
 <pinref part="R5" gate="G$1" pin="1"/>
-<wire x1="76.2" y1="144.78" x2="76.2" y2="149.86" width="0.1524" layer="91"/>
-</segment>
-</net>
-<net name="N$12" class="0">
-<segment>
-<pinref part="R6" gate="G$1" pin="1"/>
-<wire x1="96.52" y1="144.78" x2="96.52" y2="149.86" width="0.1524" layer="91"/>
-</segment>
-</net>
-<net name="N$25" class="0">
-<segment>
-<pinref part="R7" gate="G$1" pin="1"/>
-<wire x1="116.84" y1="144.78" x2="116.84" y2="149.86" width="0.1524" layer="91"/>
-</segment>
-</net>
-<net name="N$26" class="0">
-<segment>
-<pinref part="R8" gate="G$1" pin="1"/>
-<wire x1="139.7" y1="144.78" x2="139.7" y2="149.86" width="0.1524" layer="91"/>
-</segment>
-</net>
+<wire x1="76.2" y1="152.4" x2="76.2" y2="146.05" width="0.1524" layer="91"/>
+</segment>
+</net>
