File: MM_Main.sch (EAGLE design)
At the start: 67 parts, among them IC1 ULN2003AD, IC2 TB6612FNG, IC4 LD117ADT50TR, Q1 TEFT4300, Q2 TEFT4300, Q3 TEFT4300, Q4 TEFT4300, Q7 8MHz, U1 STM32F405RGT6

Commit message: rozwoj brd
Connections:
- removed net N$36: U1.PB8
- removed net N$37: U1.PB9
- new net N$42: U1.PB11
- net LED1: now also U1.PB9; no longer U1.PA12
- net LED2: now also U1.PB8; no longer U1.PA11
Changed lines of the file:
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@@
 <instance part="L1" gate="A" x="187.96" y="261.62"/>
 <instance part="L2" gate="A" x="187.96" y="241.3"/>
-<instance part="AGND8" gate="GND" x="187.96" y="25.4" rot="R270"/>
-<instance part="AGND9" gate="GND" x="187.96" y="22.86" rot="R270"/>
-<instance part="AGND10" gate="GND" x="187.96" y="20.32" rot="R270"/>
-<instance part="AGND14" gate="GND" x="187.96" y="17.78" rot="R270"/>
-<instance part="AGND16" gate="GND" x="187.96" y="15.24" rot="R270"/>
-<instance part="+3V2" gate="G$1" x="187.96" y="-68.58" rot="R90"/>
-<instance part="+3V7" gate="G$1" x="187.96" y="-71.12" rot="R90"/>
-<instance part="+3V9" gate="G$1" x="187.96" y="-73.66" rot="R90"/>
+<instance part="AGND8" gate="GND" x="185.42" y="25.4" rot="R270"/>
+<instance part="AGND9" gate="GND" x="185.42" y="22.86" rot="R270"/>
+<instance part="AGND10" gate="GND" x="185.42" y="20.32" rot="R270"/>
+<instance part="AGND14" gate="GND" x="185.42" y="17.78" rot="R270"/>
+<instance part="AGND16" gate="GND" x="185.42" y="15.24" rot="R270"/>
+<instance part="+3V2" gate="G$1" x="185.42" y="-68.58" rot="R90"/>
+<instance part="+3V7" gate="G$1" x="185.42" y="-71.12" rot="R90"/>
+<instance part="+3V9" gate="G$1" x="185.42" y="-73.66" rot="R90"/>
 <instance part="+3V15" gate="G$1" x="187.96" y="7.62" rot="R90"/>
 <instance part="AGND19" gate="GND" x="-55.88" y="259.08"/>
@@
 <pinref part="U1" gate="A" pin="VDDA"/>
 <pinref part="AGND8" gate="GND" pin="GND"/>
+<wire x1="187.96" y1="25.4" x2="190.5" y2="25.4" width="0.1524" layer="91"/>
 </segment>
 <segment>
 <pinref part="U1" gate="A" pin="VDD_2"/>
 <pinref part="AGND9" gate="GND" pin="GND"/>
+<wire x1="187.96" y1="22.86" x2="190.5" y2="22.86" width="0.1524" layer="91"/>
 </segment>
 <segment>
 <pinref part="U1" gate="A" pin="VDD_3"/>
 <pinref part="AGND10" gate="GND" pin="GND"/>
+<wire x1="187.96" y1="20.32" x2="190.5" y2="20.32" width="0.1524" layer="91"/>
 </segment>
 <segment>
 <pinref part="U1" gate="A" pin="VDD_4"/>
 <pinref part="AGND14" gate="GND" pin="GND"/>
+<wire x1="187.96" y1="17.78" x2="190.5" y2="17.78" width="0.1524" layer="91"/>
 </segment>
 <segment>
 <pinref part="U1" gate="A" pin="VDD"/>
 <pinref part="AGND16" gate="GND" pin="GND"/>
+<wire x1="187.96" y1="15.24" x2="190.5" y2="15.24" width="0.1524" layer="91"/>
 </segment>
 <segment>
@@
 <pinref part="U1" gate="A" pin="VSSA"/>
 <pinref part="+3V2" gate="G$1" pin="+3V3"/>
+<wire x1="187.96" y1="-68.58" x2="190.5" y2="-68.58" width="0.1524" layer="91"/>
 </segment>
 <segment>
 <pinref part="U1" gate="A" pin="VSS_2"/>
 <pinref part="+3V7" gate="G$1" pin="+3V3"/>
+<wire x1="187.96" y1="-71.12" x2="190.5" y2="-71.12" width="0.1524" layer="91"/>
 </segment>
 <segment>
 <pinref part="U1" gate="A" pin="VSS"/>
 <pinref part="+3V9" gate="G$1" pin="+3V3"/>
+<wire x1="187.96" y1="-73.66" x2="190.5" y2="-73.66" width="0.1524" layer="91"/>
 </segment>
 <segment>
@@
 </segment>
 <segment>
-<pinref part="U1" gate="A" pin="PA12"/>
-<wire x1="226.06" y1="-17.78" x2="231.14" y2="-17.78" width="0.1524" layer="91"/>
-<label x="231.14" y="-17.78" size="1.27" layer="95" xref="yes"/>
+<pinref part="U1" gate="A" pin="PB9"/>
+<wire x1="226.06" y1="22.86" x2="231.14" y2="22.86" width="0.1524" layer="91"/>
+<label x="231.14" y="22.86" size="1.27" layer="95" xref="yes"/>
 </segment>
 </net>
@@
 </segment>
 <segment>
-<pinref part="U1" gate="A" pin="PA11"/>
-<wire x1="226.06" y1="-20.32" x2="231.14" y2="-20.32" width="0.1524" layer="91"/>
-<label x="231.14" y="-20.32" size="1.27" layer="95" xref="yes"/>
+<pinref part="U1" gate="A" pin="PB8"/>
+<wire x1="226.06" y1="20.32" x2="231.14" y2="20.32" width="0.1524" layer="91"/>
+<label x="231.14" y="20.32" size="1.27" layer="95" xref="yes"/>
 </segment>
 </net>
@@
 </segment>
 </net>
-<net name="N$36" class="0">
-<segment>
-<pinref part="U1" gate="A" pin="PB8"/>
-<wire x1="226.06" y1="20.32" x2="228.6" y2="20.32" width="0.1524" layer="91"/>
-</segment>
-</net>
-<net name="N$37" class="0">
-<segment>
-<pinref part="U1" gate="A" pin="PB9"/>
-<wire x1="226.06" y1="22.86" x2="228.6" y2="22.86" width="0.1524" layer="91"/>
-</segment>
-</net>
 <net name="N$38" class="0">
 <segment>
@@
 </segment>
 </net>
+<net name="N$42" class="0">
+<segment>
+<pinref part="U1" gate="A" pin="PB11"/>
+<wire x1="190.5" y1="-60.96" x2="187.96" y2="-60.96" width="0.1524" layer="91"/>
+</segment>
+</net>

Commit message: aktualizacja brd
Connections:
- net GNDA: now also BAT1.1, BAT1.3
- net N$9: now also BAT1.2
Changed lines of the file:
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@@
 <part name="+3V5" library="supply1" deviceset="+3V3" device=""/>
 <part name="GND4" library="supply1" deviceset="GNDA" device=""/>
+<part name="GND5" library="supply1" deviceset="GNDA" device=""/>
+<part name="GND6" library="supply1" deviceset="GNDA" device=""/>
 </parts>
 <sheets>
@@
 <instance part="R9" gate="G$1" x="-106.68" y="129.54" rot="R90"/>
 <instance part="R17" gate="G$1" x="-106.68" y="119.38" rot="R90"/>
-<instance part="SUPPLY1" gate="G$1" x="-106.68" y="137.16"/>
+<instance part="SUPPLY1" gate="G$1" x="-106.68" y="139.7"/>
 <instance part="R18" gate="G$1" x="269.24" y="12.7"/>
 <instance part="R19" gate="G$1" x="274.32" y="7.62" rot="R90"/>
@@
 </instance>
 <instance part="GND4" gate="1" x="-152.4" y="111.76"/>
+<instance part="GND5" gate="1" x="-144.78" y="139.7"/>
+<instance part="GND6" gate="1" x="-139.7" y="139.7"/>
 </instances>
 <busses>
@@
 <pinref part="GND4" gate="1" pin="GNDA"/>
 </segment>
+<segment>
+<pinref part="BAT1" gate="A" pin="1"/>
+<pinref part="GND5" gate="1" pin="GNDA"/>
+</segment>
+<segment>
+<pinref part="BAT1" gate="A" pin="3"/>
+<pinref part="GND6" gate="1" pin="GNDA"/>
+</segment>
 </net>
 <net name="+3V3" class="0">
@@
 <pinref part="R9" gate="G$1" pin="2"/>
 <pinref part="SUPPLY1" gate="G$1" pin="+7V"/>
+<wire x1="-106.68" y1="137.16" x2="-106.68" y2="134.62" width="0.1524" layer="91"/>
 </segment>
 <segment>
@@
 <pinref part="ZAS" gate="G$1" pin="1"/>
 <wire x1="-149.86" y1="121.92" x2="-147.32" y2="121.92" width="0.1524" layer="91"/>
-</segment>
-</net>
+<pinref part="BAT1" gate="A" pin="2"/>
+<wire x1="-142.24" y1="142.24" x2="-142.24" y2="127" width="0.1524" layer="91"/>
+<wire x1="-142.24" y1="127" x2="-147.32" y2="121.92" width="0.1524" layer="91"/>
+</segment>
+</net>
