File: MM_Main.sch (EAGLE design)
At the start: 77 parts, among them IC1 ULN2003AD, IC2 TB6612FNG, IC4 LD117ADT50TR, Q1 TEFT4300, Q2 TEFT4300, Q3 TEFT4300, Q4 TEFT4300, Q5 TEFT4300, Q6 TEFT4300, Q7 8MHz

Commit message: 2 zwykle ledy z przodu
Parts:
- added LED4: green, led:LEDSML1206
- added LED6: yellow, led:LEDSML1206
- added R20, R27: 10K, resistor:R-EU_R0805
Connections:
- new net LED3: LED4.C, U$6.PB5
- new net LED5: LED6.C, U$6.PA0_AKUP
- new net LED6: U$6.PB11
- new net N$22: LED4.A, R20.1
- new net N$31: LED6.A, R27.1
- net +3V3: now also R20.2, R27.2
Other:
- note added: "po�?�?czy�? masy"
- note added: "te�? bootloader"
- note removed: "poďż˝?ďż˝?czyďż˝? masy"
- note removed: "teĹ bootloader"
- moved on the sheet: LED1, LED2, LED3, R10, R12, R13

Commit message: drc, kosmetyka, opisy, pasztet
Parts:
- renumbered BOOT0 to BT0, BOOT1 to BT1, U$4 to IC5
Changed lines of the file:
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@@
 <part name="+3V13" library="supply1" deviceset="+3V3" device=""/>
 <part name="SUPPLY5" library="supply2" deviceset="+7V" device=""/>
-<part name="BOOT1" library="GeekAmmo" deviceset="TACTILE-SWITCH" device="-7914G" value="TACTILE-SWITCH-7914G"/>
+<part name="BT1" library="GeekAmmo" deviceset="TACTILE-SWITCH" device="-7914G" value="TACTILE-SWITCH-7914G"/>
 <part name="R11" library="resistor" deviceset="R-EU_" device="R0805" value="10K"/>
 <part name="C15" library="rcl" deviceset="CPOL-EU" device="SMCD" value="tant-d-220u"/>
 <part name="GND11" library="supply1" deviceset="GNDA" device=""/>
-<part name="U$4" library="_microMouse" deviceset="MCP1825" device=""/>
+<part name="IC5" library="_microMouse" deviceset="MCP1825" device=""/>
 <part name="IC4" library="v-reg" deviceset="LD117A?*" device="DT" technology="50TR"/>
 <part name="C21" library="rcl" deviceset="CPOL-EU" device="SMCA" value="tant-a-4,7u"/>
@@
 <part name="AGND1" library="supply2" deviceset="GND" device=""/>
 <part name="JP1" library="SparkFun-Connectors" deviceset="M03" device="POLAR"/>
-<part name="BOOT0" library="GeekAmmo" deviceset="TACTILE-SWITCH" device="-7914G" value="TACTILE-SWITCH-7914G"/>
+<part name="BT0" library="GeekAmmo" deviceset="TACTILE-SWITCH" device="-7914G" value="TACTILE-SWITCH-7914G"/>
 <part name="R15" library="rcl" deviceset="R-EU_" device="R0805"/>
 <part name="D5" library="_microMouse" deviceset="SFH4545" device="-C" value="SFH4545-C"/>
@@
 <instance part="+3V13" gate="G$1" x="-185.42" y="81.28"/>
 <instance part="SUPPLY5" gate="G$1" x="-121.92" y="132.08"/>
-<instance part="BOOT1" gate="G$1" x="-63.5" y="55.88"/>
+<instance part="BT1" gate="G$1" x="-63.5" y="55.88"/>
 <instance part="R11" gate="G$1" x="-68.58" y="68.58" rot="R270"/>
 <instance part="C15" gate="G$1" x="-121.92" y="119.38"/>
 <instance part="GND11" gate="1" x="-121.92" y="111.76"/>
-<instance part="U$4" gate="G$1" x="-83.82" y="-17.78"/>
+<instance part="IC5" gate="G$1" x="-83.82" y="-17.78"/>
 <instance part="IC4" gate="G$1" x="-132.08" y="-5.08" smashed="yes">
 <attribute name="NAME" x="-139.7" y="0.762" size="1.778" layer="95"/>
@@
 <instance part="AGND1" gate="GND" x="96.52" y="-50.8"/>
 <instance part="JP1" gate="G$1" x="-149.86" y="137.16" rot="R270"/>
-<instance part="BOOT0" gate="G$1" x="205.74" y="30.48" rot="R90"/>
+<instance part="BT0" gate="G$1" x="205.74" y="30.48" rot="R90"/>
 <instance part="R15" gate="G$1" x="86.36" y="154.94" rot="R90"/>
 <instance part="D5" gate="G$1" x="86.36" y="144.78"/>
@@
 </segment>
 <segment>
-<pinref part="U$4" gate="G$1" pin="GND"/>
+<pinref part="IC5" gate="G$1" pin="GND"/>
 <wire x1="-96.52" y1="-17.78" x2="-111.76" y2="-17.78" width="0.1524" layer="91"/>
 <wire x1="-111.76" y1="-17.78" x2="-111.76" y2="-15.24" width="0.1524" layer="91"/>
@@
 </segment>
 <segment>
-<pinref part="U$4" gate="G$1" pin="OUT"/>
+<pinref part="IC5" gate="G$1" pin="OUT"/>
 <pinref part="R16" gate="G$1" pin="2"/>
 <wire x1="-68.58" y1="-12.7" x2="-60.96" y2="-12.7" width="0.1524" layer="91"/>
@@
 <wire x1="193.04" y1="35.56" x2="193.04" y2="33.02" width="0.1524" layer="91"/>
 <wire x1="205.74" y1="35.56" x2="193.04" y2="35.56" width="0.1524" layer="91"/>
-<pinref part="BOOT0" gate="G$1" pin="3"/>
+<pinref part="BT0" gate="G$1" pin="3"/>
 </segment>
 <segment>
@@
 <net name="N$29" class="0">
 <segment>
-<pinref part="BOOT1" gate="G$1" pin="1"/>
+<pinref part="BT1" gate="G$1" pin="1"/>
 <pinref part="R11" gate="G$1" pin="2"/>
 <wire x1="-68.58" y1="55.88" x2="-68.58" y2="63.5" width="0.1524" layer="91"/>
@@
 <net name="N$1" class="0">
 <segment>
-<pinref part="U$4" gate="G$1" pin="PWRGD"/>
+<pinref part="IC5" gate="G$1" pin="PWRGD"/>
 <pinref part="R16" gate="G$1" pin="1"/>
 <wire x1="-68.58" y1="-22.86" x2="-60.96" y2="-22.86" width="0.1524" layer="91"/>
@@
 <net name="+5V" class="0">
 <segment>
-<pinref part="U$4" gate="G$1" pin="SHDN"/>
+<pinref part="IC5" gate="G$1" pin="SHDN"/>
 <wire x1="-96.52" y1="-22.86" x2="-99.06" y2="-22.86" width="0.1524" layer="91"/>
-<pinref part="U$4" gate="G$1" pin="IN"/>
+<pinref part="IC5" gate="G$1" pin="IN"/>
 <wire x1="-96.52" y1="-12.7" x2="-99.06" y2="-12.7" width="0.1524" layer="91"/>
 <wire x1="-99.06" y1="-12.7" x2="-104.14" y2="-12.7" width="0.1524" layer="91"/>
@@
 <wire x1="205.74" y1="20.32" x2="190.5" y2="20.32" width="0.1524" layer="91"/>
 <wire x1="205.74" y1="25.4" x2="205.74" y2="20.32" width="0.1524" layer="91"/>
-<pinref part="BOOT0" gate="G$1" pin="1"/>
+<pinref part="BT0" gate="G$1" pin="1"/>
 </segment>
 </net>
@@
 <net name="BTN" class="0">
 <segment>
-<pinref part="BOOT1" gate="G$1" pin="3"/>
+<pinref part="BT1" gate="G$1" pin="3"/>
 <wire x1="-58.42" y1="55.88" x2="-55.88" y2="55.88" width="0.1524" layer="91"/>
 <label x="-53.34" y="55.88" size="1.27" layer="95" xref="yes"/>

Commit message: poprawa bledow, dodanie rezystorow na wyjsciach stm-glownie w modolach, poprawa elementu 9axis z biblioteki
Parts:
- added R26: 10K, resistor:R-EU_R0805
Connections:
- new net N$26: R26.1, SV1.8
- net BT_RXD: now also R26.2; no longer SV1.6
- net BT_TXD: now also SV1.6; no longer SV1.8
- net INT_A: now also U$1.INT_A; no longer U$1.INT_G
- net SCLK: now also U$1.CLK; no longer U$1.SCLK
Other:
- note added: "GND"
- note added: "HC-06"
- note added: "Rx"
- note added: "Tx"
- note added: "VCC"
Changed lines of the file:
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@@
 <part name="ZAS" library="special" deviceset="SW_DIP-1" device=""/>
 <part name="FUSE" library="resistor" deviceset="R-EU_" device="M2012"/>
-<part name="+3V3" library="supply1" deviceset="+3V3" device=""/>
-<part name="AGND7" library="supply2" deviceset="GND" device=""/>
 <part name="U$2" library="_microMouse" deviceset="LI-POL" device="-DUALKSY_220MAH_D" value="LI-POL-DUALKSY_220MAH_D"/>
 <part name="U$1" library="_microMouse" deviceset="9AXIS_MODULE" device=""/>
@@
 <part name="LED6" library="led" deviceset="LED" device="SML1206" value="yellow"/>
 <part name="+3V29" library="supply1" deviceset="+3V3" device=""/>
+<part name="R26" library="resistor" deviceset="R-EU_" device="R0805" value="10K"/>
 </parts>
 <sheets>
@@
 <text x="40.64" y="73.66" size="1.27" layer="91">PA2 i PA3</text>
 <text x="27.94" y="147.32" size="1.778" layer="91">TODO: sprawdzic kolejnosc ledow</text>
+<text x="-187.96" y="33.02" size="1.27" layer="91">Rx</text>
+<text x="-187.96" y="30.48" size="1.27" layer="91">Tx</text>
+<text x="-187.96" y="27.94" size="1.27" layer="91">GND</text>
+<text x="-187.96" y="25.4" size="1.27" layer="91">VCC</text>
+<text x="-185.42" y="38.1" size="1.27" layer="91" rot="R180">HC-06</text>
 </plain>
 <instances>
@@
 <instance part="ZAS" gate="G$1" x="-139.7" y="121.92" rot="R180"/>
 <instance part="FUSE" gate="G$1" x="-127" y="121.92" rot="R180"/>
-<instance part="+3V3" gate="G$1" x="337.82" y="78.74" rot="MR270"/>
-<instance part="AGND7" gate="GND" x="337.82" y="76.2" rot="MR90"/>
 <instance part="U$2" gate="G$1" x="-71.12" y="121.92"/>
 <instance part="U$1" gate="G$1" x="358.14" y="76.2"/>
@@
 <instance part="LED6" gate="G$1" x="-101.6" y="58.42"/>
 <instance part="+3V29" gate="G$1" x="-101.6" y="81.28"/>
+<instance part="R26" gate="G$1" x="-165.1" y="33.02" rot="R180"/>
 </instances>
 <busses>
@@
 </segment>
 <segment>
-<wire x1="342.9" y1="76.2" x2="340.36" y2="76.2" width="0.1524" layer="91"/>
-<pinref part="AGND7" gate="GND" pin="GND"/>
-<pinref part="U$1" gate="G$1" pin="GND"/>
-</segment>
-<segment>
 <wire x1="-10.16" y1="22.86" x2="-10.16" y2="25.4" width="0.1524" layer="91"/>
 <pinref part="C_VSSA" gate="G$1" pin="2"/>
@@
 <pinref part="AGND4" gate="GND" pin="GND"/>
 </segment>
+<segment>
+<pinref part="U$1" gate="G$1" pin="GND"/>
+<wire x1="342.9" y1="73.66" x2="340.36" y2="73.66" width="0.1524" layer="91"/>
+<label x="340.36" y="73.66" size="1.27" layer="95" rot="R180" xref="yes"/>
+</segment>
 </net>
 <net name="MOSI" class="0">
-<segment>
-<wire x1="373.38" y1="76.2" x2="386.08" y2="76.2" width="0.1524" layer="91"/>
-<label x="386.08" y="76.2" size="1.27" layer="95" rot="MR180" xref="yes"/>
-<pinref part="U$1" gate="G$1" pin="MOSI"/>
-</segment>
 <segment>
 <wire x1="454.66" y1="5.08" x2="459.74" y2="5.08" width="0.1524" layer="91"/>
@@
 <pinref part="U$6" gate="G$1" pin="PC12"/>
 </segment>
+<segment>
+<pinref part="U$1" gate="G$1" pin="MOSI"/>
+<wire x1="373.38" y1="76.2" x2="375.92" y2="76.2" width="0.1524" layer="91"/>
+<label x="375.92" y="76.2" size="1.27" layer="95" xref="yes"/>
+</segment>
 </net>
 <net name="MISO" class="0">
-<segment>
-<wire x1="373.38" y1="81.28" x2="386.08" y2="81.28" width="0.1524" layer="91"/>
-<label x="386.08" y="81.28" size="1.27" layer="95" rot="MR180" xref="yes"/>
-<pinref part="U$1" gate="G$1" pin="MISO"/>
-</segment>
 <segment>
 <wire x1="454.66" y1="2.54" x2="459.74" y2="2.54" width="0.1524" layer="91"/>
@@
 <pinref part="U$6" gate="G$1" pin="PC11"/>
 </segment>
+<segment>
+<pinref part="U$1" gate="G$1" pin="MISO"/>
+<wire x1="373.38" y1="78.74" x2="375.92" y2="78.74" width="0.1524" layer="91"/>
+<label x="375.92" y="78.74" size="1.27" layer="95" xref="yes"/>
+</segment>
 </net>
 <net name="SCLK" class="0">
-<segment>
-<wire x1="373.38" y1="73.66" x2="386.08" y2="73.66" width="0.1524" layer="91"/>
-<label x="386.08" y="73.66" size="1.27" layer="95" rot="MR180" xref="yes"/>
-<pinref part="U$1" gate="G$1" pin="SCLK"/>
-</segment>
 <segment>
 <wire x1="454.66" y1="0" x2="459.74" y2="0" width="0.1524" layer="91"/>
@@
 <label x="48.26" y="15.24" size="1.016" layer="95" rot="R180" xref="yes"/>
 <pinref part="U$6" gate="G$1" pin="PC10"/>
+</segment>
+<segment>
+<pinref part="U$1" gate="G$1" pin="CLK"/>
+<wire x1="373.38" y1="73.66" x2="375.92" y2="73.66" width="0.1524" layer="91"/>
+<label x="375.92" y="73.66" size="1.27" layer="95" xref="yes"/>
 </segment>
 </net>
@@
 </segment>
 <segment>
-<wire x1="342.9" y1="78.74" x2="340.36" y2="78.74" width="0.1524" layer="91"/>
-<pinref part="+3V3" gate="G$1" pin="+3V3"/>
-<pinref part="U$1" gate="G$1" pin="+3V3"/>
-</segment>
-<segment>
 <wire x1="-10.16" y1="33.02" x2="-10.16" y2="35.56" width="0.1524" layer="91"/>
 <wire x1="-10.16" y1="35.56" x2="-2.54" y2="35.56" width="0.1524" layer="91"/>
@@
 <wire x1="-101.6" y1="78.74" x2="-101.6" y2="76.2" width="0.1524" layer="91"/>
 </segment>
+<segment>
+<pinref part="U$1" gate="G$1" pin="+3V3"/>
+<wire x1="342.9" y1="81.28" x2="340.36" y2="81.28" width="0.1524" layer="91"/>
+<label x="340.36" y="81.28" size="1.27" layer="95" rot="R180" xref="yes"/>
+</segment>
 </net>
 <net name="+7V" class="0">
@@
 </segment>
 <segment>
-<wire x1="-160.02" y1="33.02" x2="-162.56" y2="33.02" width="0.1524" layer="91"/>
-<label x="-162.56" y="33.02" size="1.016" layer="95" rot="R180" xref="yes"/>
-<pinref part="SV1" gate="G$1" pin="8"/>
+<pinref part="SV1" gate="G$1" pin="6"/>
+<wire x1="-160.02" y1="30.48" x2="-172.72" y2="30.48" width="0.1524" layer="91"/>
+<label x="-172.72" y="30.48" size="1.27" layer="95" rot="R180" xref="yes"/>
 </segment>
 </net>
@@
 </segment>
 <segment>
-<wire x1="-160.02" y1="30.48" x2="-162.56" y2="30.48" width="0.1524" layer="91"/>
-<label x="-162.56" y="30.48" size="1.016" layer="95" rot="R180" xref="yes"/>
-<pinref part="SV1" gate="G$1" pin="6"/>
+<pinref part="R26" gate="G$1" pin="2"/>
+<wire x1="-170.18" y1="33.02" x2="-172.72" y2="33.02" width="0.1524" layer="91"/>
+<label x="-172.72" y="33.02" size="1.27" layer="95" rot="R180" xref="yes"/>
 </segment>
 </net>
@@
 <net name="CS_G" class="0">
 <segment>
-<wire x1="373.38" y1="78.74" x2="386.08" y2="78.74" width="0.1524" layer="91"/>
-<label x="386.08" y="78.74" size="1.27" layer="95" rot="MR180" xref="yes"/>
-<pinref part="U$1" gate="G$1" pin="CS_G"/>
-</segment>
-<segment>
 <wire x1="454.66" y1="10.16" x2="459.74" y2="10.16" width="0.1524" layer="91"/>
 <label x="459.74" y="10.16" size="1.27" layer="95" xref="yes"/>
@@
 <pinref part="U$6" gate="G$1" pin="PB3"/>
 </segment>
+<segment>
+<pinref part="U$1" gate="G$1" pin="CS_G"/>
+<wire x1="373.38" y1="81.28" x2="375.92" y2="81.28" width="0.1524" layer="91"/>
+<label x="375.92" y="81.28" size="1.27" layer="95" xref="yes"/>
+</segment>
 </net>
 <net name="CS_A" class="0">
-<segment>
-<wire x1="342.9" y1="73.66" x2="330.2" y2="73.66" width="0.1524" layer="91"/>
-<label x="330.2" y="73.66" size="1.27" layer="95" rot="MR0" xref="yes"/>
-<pinref part="U$1" gate="G$1" pin="CS_A"/>
-</segment>
 <segment>
 <wire x1="454.66" y1="12.7" x2="459.74" y2="12.7" width="0.1524" layer="91"/>
@@
 <label x="48.26" y="2.54" size="1.016" layer="95" rot="R180" xref="yes"/>
 <pinref part="U$6" gate="G$1" pin="PB4"/>
+</segment>
+<segment>
+<pinref part="U$1" gate="G$1" pin="CS_A"/>
+<wire x1="342.9" y1="78.74" x2="340.36" y2="78.74" width="0.1524" layer="91"/>
+<label x="340.36" y="78.74" size="1.27" layer="95" rot="R180" xref="yes"/>
 </segment>
 </net>
@@
 </segment>
 <segment>
-<wire x1="342.9" y1="81.28" x2="330.2" y2="81.28" width="0.1524" layer="91"/>
-<label x="330.2" y="81.28" size="1.27" layer="95" rot="MR0" xref="yes"/>
-<pinref part="U$1" gate="G$1" pin="INT_G"/>
-</segment>
-<segment>
 <pinref part="U$6" gate="G$1" pin="PB0"/>
 <wire x1="124.46" y1="5.08" x2="127" y2="5.08" width="0.1524" layer="91"/>
 <label x="127" y="5.08" size="1.27" layer="95" xref="yes"/>
+</segment>
+<segment>
+<pinref part="U$1" gate="G$1" pin="INT_A"/>
+<wire x1="342.9" y1="76.2" x2="340.36" y2="76.2" width="0.1524" layer="91"/>
+<label x="340.36" y="76.2" size="1.27" layer="95" rot="R180" xref="yes"/>
 </segment>
 </net>
@@
 </segment>
 </net>
+<net name="N$25" class="0">
+<segment>
+<wire x1="-190.5" y1="35.56" x2="-190.5" y2="22.86" width="0.1524" layer="91"/>
+<wire x1="-190.5" y1="35.56" x2="-185.42" y2="35.56" width="0.1524" layer="91"/>
+<wire x1="-190.5" y1="22.86" x2="-185.42" y2="22.86" width="0.1524" layer="91"/>
+</segment>
+</net>
+<net name="N$26" class="0">
+<segment>
+<pinref part="SV1" gate="G$1" pin="8"/>
+<pinref part="R26" gate="G$1" pin="1"/>
+</segment>
+</net>

Commit message: pixi
Parts:
- R26: value 10K -> (none); device resistor:R-EU_R0805 -> rcl:R-EU_R0805
Connections:
- net BT_RXD: now also SV1.8; no longer R26.2
- net BT_TXD: now also R26.2; no longer SV1.6
- net N$26: now also SV1.6; no longer SV1.8
Other:
- moved on the sheet: LED6, R26, R27
Changed lines of the file:
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@@
 <part name="LED6" library="led" deviceset="LED" device="SML1206" value="yellow"/>
 <part name="+3V29" library="supply1" deviceset="+3V3" device=""/>
-<part name="R26" library="resistor" deviceset="R-EU_" device="R0805" value="10K"/>
+<part name="R26" library="rcl" deviceset="R-EU_" device="R0805"/>
 </parts>
 <sheets>
@@
 <instance part="R20" gate="G$1" x="-142.24" y="71.12" rot="R90"/>
 <instance part="+3V14" gate="G$1" x="-142.24" y="81.28"/>
-<instance part="R27" gate="G$1" x="-101.6" y="71.12" rot="R90"/>
-<instance part="LED6" gate="G$1" x="-101.6" y="58.42"/>
-<instance part="+3V29" gate="G$1" x="-101.6" y="81.28"/>
-<instance part="R26" gate="G$1" x="-165.1" y="33.02" rot="R180"/>
+<instance part="R27" gate="G$1" x="-119.38" y="71.12" rot="R90"/>
+<instance part="LED6" gate="G$1" x="-119.38" y="58.42"/>
+<instance part="+3V29" gate="G$1" x="-119.38" y="81.28"/>
+<instance part="R26" gate="G$1" x="-165.1" y="30.48" rot="R180"/>
 </instances>
 <busses>
@@
 <pinref part="+3V29" gate="G$1" pin="+3V3"/>
 <pinref part="R27" gate="G$1" pin="2"/>
-<wire x1="-101.6" y1="78.74" x2="-101.6" y2="76.2" width="0.1524" layer="91"/>
+<wire x1="-119.38" y1="78.74" x2="-119.38" y2="76.2" width="0.1524" layer="91"/>
 </segment>
 <segment>
@@
 </segment>
 <segment>
-<wire x1="73.66" y1="38.1" x2="73.66" y2="40.64" width="0.1524" layer="91"/>
+<wire x1="73.66" y1="38.1" x2="73.66" y2="43.18" width="0.1524" layer="91"/>
 <pinref part="U$6" gate="G$1" pin="PA13"/>
+<label x="73.66" y="43.18" size="1.27" layer="95" rot="R90" xref="yes"/>
 </segment>
 <segment>
@@
 </segment>
 <segment>
-<pinref part="SV1" gate="G$1" pin="6"/>
-<wire x1="-160.02" y1="30.48" x2="-172.72" y2="30.48" width="0.1524" layer="91"/>
+<pinref part="R26" gate="G$1" pin="2"/>
+<wire x1="-170.18" y1="30.48" x2="-172.72" y2="30.48" width="0.1524" layer="91"/>
 <label x="-172.72" y="30.48" size="1.27" layer="95" rot="R180" xref="yes"/>
 </segment>
@@
 </segment>
 <segment>
-<pinref part="R26" gate="G$1" pin="2"/>
-<wire x1="-170.18" y1="33.02" x2="-172.72" y2="33.02" width="0.1524" layer="91"/>
 <label x="-172.72" y="33.02" size="1.27" layer="95" rot="R180" xref="yes"/>
+<pinref part="SV1" gate="G$1" pin="8"/>
+<wire x1="-172.72" y1="33.02" x2="-160.02" y2="33.02" width="0.1524" layer="91"/>
 </segment>
 </net>
@@
 <wire x1="101.6" y1="38.1" x2="101.6" y2="40.64" width="0.1524" layer="91"/>
 <pinref part="U$6" gate="G$1" pin="PB14"/>
+<label x="101.6" y="40.64" size="1.27" layer="95" rot="R90" xref="yes"/>
 </segment>
 </net>
@@
 <wire x1="99.06" y1="38.1" x2="99.06" y2="40.64" width="0.1524" layer="91"/>
 <pinref part="U$6" gate="G$1" pin="PB15"/>
+<label x="99.06" y="40.64" size="1.27" layer="95" rot="R90" xref="yes"/>
 </segment>
 </net>
@@
 <wire x1="96.52" y1="38.1" x2="96.52" y2="40.64" width="0.1524" layer="91"/>
 <pinref part="U$6" gate="G$1" pin="PC6"/>
+<label x="96.52" y="40.64" size="1.27" layer="95" rot="R90" xref="yes"/>
 </segment>
 </net>
@@
 <wire x1="78.74" y1="7.62" x2="78.74" y2="-7.62" width="0.1524" layer="91"/>
 <wire x1="78.74" y1="-7.62" x2="50.8" y2="-7.62" width="0.1524" layer="91"/>
+<label x="50.8" y="7.62" size="1.27" layer="95" rot="R180" xref="yes"/>
 </segment>
 </net>
@@
 <segment>
 <pinref part="LED6" gate="G$1" pin="C"/>
-<wire x1="-101.6" y1="53.34" x2="-101.6" y2="50.8" width="0.1524" layer="91"/>
-<wire x1="-101.6" y1="50.8" x2="-93.98" y2="50.8" width="0.1524" layer="91"/>
-<label x="-93.98" y="50.8" size="1.27" layer="95" xref="yes"/>
+<wire x1="-119.38" y1="53.34" x2="-119.38" y2="50.8" width="0.1524" layer="91"/>
+<wire x1="-119.38" y1="50.8" x2="-111.76" y2="50.8" width="0.1524" layer="91"/>
+<label x="-111.76" y="50.8" size="1.27" layer="95" xref="yes"/>
 </segment>
 <segment>
 <pinref part="U$6" gate="G$1" pin="PA0_AKUP"/>
 <wire x1="101.6" y1="-35.56" x2="101.6" y2="-38.1" width="0.1524" layer="91"/>
+<label x="101.6" y="-38.1" size="1.27" layer="95" rot="R270" xref="yes"/>
 </segment>
 </net>
@@
 <pinref part="R27" gate="G$1" pin="1"/>
 <pinref part="LED6" gate="G$1" pin="A"/>
-<wire x1="-101.6" y1="66.04" x2="-101.6" y2="60.96" width="0.1524" layer="91"/>
+<wire x1="-119.38" y1="66.04" x2="-119.38" y2="60.96" width="0.1524" layer="91"/>
 </segment>
 </net>
@@
 <net name="N$26" class="0">
 <segment>
-<pinref part="SV1" gate="G$1" pin="8"/>
+<pinref part="SV1" gate="G$1" pin="6"/>
 <pinref part="R26" gate="G$1" pin="1"/>
 </segment>

Commit message: poprawki warst opisowych, dodanie gerberow mm
Parts:
- removed U$2: LI-POL-DUALKSY_220MAH_D, _microMouse:LI-POL-DUALKSY_220MAH_D
Changed lines of the file:
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@@
 <part name="ZAS" library="special" deviceset="SW_DIP-1" device=""/>
 <part name="FUSE" library="resistor" deviceset="R-EU_" device="M2012"/>
-<part name="U$2" library="_microMouse" deviceset="LI-POL" device="-DUALKSY_220MAH_D" value="LI-POL-DUALKSY_220MAH_D"/>
 <part name="U$1" library="_microMouse" deviceset="9AXIS_MODULE" device=""/>
 <part name="+3V1" library="supply1" deviceset="+3V3" device=""/>
@@
 <instance part="ZAS" gate="G$1" x="-139.7" y="121.92" rot="R180"/>
 <instance part="FUSE" gate="G$1" x="-127" y="121.92" rot="R180"/>
-<instance part="U$2" gate="G$1" x="-71.12" y="121.92"/>
 <instance part="U$1" gate="G$1" x="358.14" y="76.2"/>
 <instance part="+3V1" gate="G$1" x="-12.7" y="40.64"/>
