File: gyro.brd (EAGLE design)
At the start: 27.9 x 15.2 mm, 16 parts, among them IC3 FXAS21002C

Commit message: gerbery
Changed lines of the file:
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@@
 <layer number="14" name="Route14" color="1" fill="6" visible="no" active="no"/>
 <layer number="15" name="Route15" color="4" fill="6" visible="no" active="no"/>
-<layer number="16" name="Bottom" color="1" fill="1" visible="yes" active="yes"/>
+<layer number="16" name="Bottom" color="1" fill="1" visible="no" active="yes"/>
 <layer number="17" name="Pads" color="2" fill="1" visible="yes" active="yes"/>
 <layer number="18" name="Vias" color="2" fill="1" visible="yes" active="yes"/>
-<layer number="19" name="Unrouted" color="6" fill="1" visible="yes" active="yes"/>
+<layer number="19" name="Unrouted" color="6" fill="1" visible="no" active="yes"/>
 <layer number="20" name="Dimension" color="15" fill="1" visible="yes" active="yes"/>
 <layer number="21" name="tPlace" color="7" fill="1" visible="yes" active="yes"/>
 <layer number="22" name="bPlace" color="7" fill="1" visible="yes" active="yes"/>
-<layer number="23" name="tOrigins" color="15" fill="1" visible="yes" active="yes"/>
-<layer number="24" name="bOrigins" color="15" fill="1" visible="yes" active="yes"/>
+<layer number="23" name="tOrigins" color="15" fill="1" visible="no" active="yes"/>
+<layer number="24" name="bOrigins" color="15" fill="1" visible="no" active="yes"/>
 <layer number="25" name="tNames" color="7" fill="1" visible="yes" active="yes"/>
-<layer number="26" name="bNames" color="7" fill="1" visible="yes" active="yes"/>
+<layer number="26" name="bNames" color="7" fill="1" visible="no" active="yes"/>
 <layer number="27" name="tValues" color="7" fill="1" visible="no" active="yes"/>
 <layer number="28" name="bValues" color="7" fill="1" visible="no" active="yes"/>
@@
 <wire x1="17.6784" y1="94.9424" x2="17.6784" y2="96.0882" width="0.254" layer="1"/>
 <wire x1="21.4699" y1="94.9339" x2="21.4699" y2="95.4971" width="0.254" layer="1"/>
-<wire x1="21.4699" y1="95.4971" x2="20.8788" y2="96.0882" width="0.254" layer="1"/>
+<wire x1="21.4699" y1="95.4971" x2="21.1328" y2="95.8342" width="0.254" layer="1"/>
 <wire x1="12.1302" y1="91.6528" x2="12.1302" y2="90.7508" width="0.254" layer="1"/>
 <wire x1="12.1302" y1="90.7508" x2="12.254" y2="90.627" width="0.254" layer="1"/>

Commit message: zamiana warstw
Other:
- board text added: "C1"
- board text added: "C10"
- board text added: "C2"
- board text added: "C3"
- board text added: "C4"
- board text added: "C5"
- board text added: "C9"
- board text added: "INT_G"
- board text added: "R1"
- board text added: "R2"
- board text added: "R3"
- board text added: "R4"
